File: driver/motherboard-v4/motherboard.kicad_pcb (KiCad board)
At the start: 2 copper layers, 88.9 x 48.3 mm, 1 part

Commit message: Add motherboard fritzing.
Parts:
- removed A1: RaspberryPi_Pico_W, Module:RaspberryPi_Pico_W_SMD
- added U1: Raspberry Pi Pico 2 W, Module:RaspberryPi_Pico_W_SMD, F.Cu at (69.8, 54.6)
Routing:
- net Net-(A1-GND-Pad13): track 167.6 -> 0.00 mm, vias 93 -> 0
- net (no net): track 439.4 -> 561.3 mm, vias 243 -> 315
- net unconnected-(A1-GPIO0-Pad1): track 68.6 -> 0.00 mm, vias 41 -> 0
- net unconnected-(A1-GPIO1-Pad2): track 63.5 -> 0.00 mm, vias 38 -> 0
- net unconnected-(U1-GP27-Pad32): track 0.00 -> 45.7 mm, vias 0 -> 21
- net unconnected-(U1-GP0-Pad1): track 0.00 -> 33.0 mm, vias 0 -> 20
- net unconnected-(U1-GP1-Pad2): track 0.00 -> 25.4 mm, vias 0 -> 15
- net unconnected-(U1-GP8-Pad11): track 0.00 -> 20.3 mm, vias 0 -> 12
- net unconnected-(U1-GP7-Pad10): track 0.00 -> 20.3 mm, vias 0 -> 12
- net unconnected-(U1-GP6-Pad9): track 0.00 -> 20.3 mm, vias 0 -> 12
- net unconnected-(U1-GP5-Pad7): track 0.00 -> 20.3 mm, vias 0 -> 12
- net unconnected-(U1-GND-Pad8): track 0.00 -> 20.3 mm, vias 0 -> 12
- net unconnected-(U1-GND-Pad3): track 0.00 -> 20.3 mm, vias 0 -> 12
- net unconnected-(A1-GPIO6-Pad9): track 20.3 -> 0.00 mm, vias 12 -> 0
- net unconnected-(A1-GPIO5-Pad7): track 20.3 -> 0.00 mm, vias 12 -> 0
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